Commit message: added physics to urdf

File: urdf/scout.urdf (robot description, URDF)
Before this commit: robot scout_rover, 2 links, 1 joints
Links:
- added link camera_link, mass 0.1; collision box size=0.05 0.05 0.05; visual box size=0.05 0.05 0.05
- added link camera_link_optical
- added link caster_wheel, mass 0.5; collision sphere radius=0.05; visual sphere radius=0.05
- added link left_wheel, mass 1.0; collision cylinder length=0.05 radius=0.1; visual cylinder length=0.05 radius=0.1
- link base_link: mass None -> 5.0; geometry collision box size=0.4 0.3 0.1; visual box size=0.4 0.3 0.1
- link right_wheel: mass None -> 1.0; geometry collision cylinder length=0.05 radius=0.1; visual cylinder length=0.05 radius=0.1
Joints:
- added joint base_to_camera: type fixed, parent base_link, child camera_link, origin xyz=0.2 0.0 0.05 rpy=0 0 0
- added joint base_to_caster: type fixed, parent base_link, child caster_wheel, origin xyz=-0.15 0.0 -0.05 rpy=0 0 0
- added joint base_to_left_wheel: type continuous, parent base_link, child left_wheel, origin xyz=0.15 0.175 0.0 rpy=-1.5708 0 0, axis 0 0 1
- added joint camera_optical_joint: type fixed, parent camera_link, child camera_link_optical, origin xyz=0 0 0 rpy=-1.5708 0 -1.5708
